File: eth_poe.sch (KiCad schematic (older format))
At the start: 42 parts, among them J101 HR861153C, U105 W5500, Y101 25MHz

Commit message: Minor cleanup
Parts:
- U105: symbol SD1-rescue:W5500-Interface_Ethernet -> Interface_Ethernet:W5500
Changed lines of the file:
@@
 	7200 4300 7200 4400
 $Comp
-L SD1-rescue:W5500-Interface_Ethernet U105
+L Interface_Ethernet:W5500 U105
 U 1 1 5FAC6941
 P 7100 3100

Commit message: Added CO sensor
Carbon Monoxide Sensor layout
Parts:
- U105: symbol Interface_Ethernet:W5500 -> SD1-rescue:W5500-Interface_Ethernet
Changed lines of the file:
@@
 	7200 4300 7200 4400
 $Comp
-L Interface_Ethernet:W5500 U105
+L SD1-rescue:W5500-Interface_Ethernet U105
 U 1 1 5FAC6941
 P 7100 3100
