File: eth_poe.sch (KiCad schematic (older format))
At the start: 42 parts, among them J101 HR861153C, U105 W5500, Y101 25MHz

Commit message: Continue part picking
Parts:
- C122: Digikey (none) -> 1276-CL10B223KC8WPNCCT-ND; Error (none) -> 10%; LCSC (none) -> C472763; MPN (none) -> CL10B223KC8WPNC; Note (none) -> CAP CER 22NF X7R 50V 0603
- C123, C124: Digikey (none) -> 311-1084-1-ND; LCSC (none) -> C107097; MPN (none) -> CC0603KRX7R9BB682; Note (none) -> CAP CER 6800PF 50V X7R 0603
- C125: value 10n -> 8.2nF; Alt (none) -> CAP CER 6800PF 50V X7R 0603; Current (none) -> CAP CER 6800PF 50V X7R 0603; Description (none) -> CAP CER 6800PF 50V X7R 0603; Digikey (none) -> 311-1811-1-ND; Error (none) -> CAP CER 6800PF 50V X7R 0603; LCSC (none) -> C113812; MPN (none) -> CC0603KRX7R9BB822; Mfr (none) -> CAP CER 6800PF 50V X7R 0603; Note (none) -> CAP CER 8.2NF X7R 50V 0603
- C129: footprint Capacitor_SMD:C_1206_3216Metric -> Capacitor_SMD:C_0603_1608Metric; Digikey (none) -> 399-3482-1-ND; LCSC (none) -> C86016; MPN (none) -> C0603C475K9PACTU; Note (none) -> CAP CER 4.7UF 6.3V X5R 0603
- FB101: value 470 -> Ferrite_Bead_Small; Alt (none) -> Ferrite_Bead_Small; Current 490-5223-1-ND -> Ferrite_Bead_Small; Description BLM18PG471SN1D -> Ferrite_Bead_Small; Error 470 Ohms @ 100MHz 1 Power Line Ferrite Bead 0603 1A 200mOhm -> Ferrite_Bead_Small; LCSC Ferrite_Bead_Small -> C97853; Mfr (none) -> 470 Ohms @ 100MHz 1 Power Line Ferrite Bead 0603 1A 200mOhm
Changed lines of the file:
@@
 AR Path="/5F9D72A5/5FAC68EB" Ref="C?"  Part="1"
 AR Path="/5FCEDB09/5FAC68EB" Ref="C160"  Part="1"
-F 0 "C160" V 3700 3500 50  0000 R CNN
-F 1 "10n" V 3700 3650 50  0000 C CNN
+F 0 "C160" V 3521 3550 50  0000 C CNN
+F 1 "8.2nF" V 3612 3550 50  0000 C CNN
 F 2 "Capacitor_SMD:C_0603_1608Metric" H 3750 3550 50  0001 C CNN
-F 3 "~" H 3750 3550 50  0001 C CNN
+F 3 "CAP CER 6800PF 50V X7R 0603" H 3750 3550 50  0001 C CNN
+F 4 "CAP CER 6800PF 50V X7R 0603" H 3750 3550 50  0001 C CNN "Alt"
+F 5 "CAP CER 6800PF 50V X7R 0603" H 3750 3550 50  0001 C CNN "Current"
+F 6 "CAP CER 6800PF 50V X7R 0603" H 3750 3550 50  0001 C CNN "Description"
+F 7 "311-1811-1-ND" H 3750 3550 50  0001 C CNN "Digikey"
+F 8 "CAP CER 6800PF 50V X7R 0603" H 3750 3550 50  0001 C CNN "Error"
+F 9 "C113812" H 3750 3550 50  0001 C CNN "LCSC"
+F 10 "CC0603KRX7R9BB822" H 3750 3550 50  0001 C CNN "MPN"
+F 11 "CAP CER 6800PF 50V X7R 0603" H 3750 3550 50  0001 C CNN "Mfr"
+F 12 "CAP CER 8.2NF X7R 50V 0603" H 3750 3550 50  0001 C CNN "Note"
 	1    3750 3550
 	0    -1   1    0
@@
 F 2 "Capacitor_SMD:C_0603_1608Metric" H 2600 3000 50  0001 C CNN
 F 3 "~" H 2600 3000 50  0001 C CNN
+F 4 "311-1084-1-ND" H 2600 3000 50  0001 C CNN "Digikey"
+F 5 "C107097" H 2600 3000 50  0001 C CNN "LCSC"
+F 6 "CC0603KRX7R9BB682" H 2600 3000 50  0001 C CNN "MPN"
+F 7 "CAP CER 6800PF 50V X7R 0603" H 2600 3000 50  0001 C CNN "Note"
 	1    2600 3000
 	0    -1   1    0
@@
 F 2 "Capacitor_SMD:C_0603_1608Metric" H 2600 2600 50  0001 C CNN
 F 3 "~" H 2600 2600 50  0001 C CNN
+F 4 "311-1084-1-ND" H 2600 2600 50  0001 C CNN "Digikey"
+F 5 "C107097" H 2600 2600 50  0001 C CNN "LCSC"
+F 6 "CC0603KRX7R9BB682" H 2600 2600 50  0001 C CNN "MPN"
+F 7 "CAP CER 6800PF 50V X7R 0603" H 2600 2600 50  0001 C CNN "Note"
 	1    2600 2600
 	0    -1   1    0
@@
 F 2 "Capacitor_SMD:C_0603_1608Metric" H 3050 2300 50  0001 C CNN
 F 3 "~" H 3050 2300 50  0001 C CNN
+F 4 "1276-CL10B223KC8WPNCCT-ND" H 3050 2300 50  0001 C CNN "Digikey"
+F 5 "10%" H 3050 2300 50  0001 C CNN "Error"
+F 6 "C472763" H 3050 2300 50  0001 C CNN "LCSC"
+F 7 "CL10B223KC8WPNC" H 3050 2300 50  0001 C CNN "MPN"
+F 8 "CAP CER 22NF X7R 50V 0603" H 3050 2300 50  0001 C CNN "Note"
 	1    3050 2300
 	0    -1   1    0
@@
 AR Path="/5FCEDB09/5FAC6A06" Ref="FB101"  Part="1"
 F 0 "FB101" V 7000 1500 50  0000 C CNN
-F 1 "470" V 6954 1250 50  0001 C CNN
+F 1 "Ferrite_Bead_Small" V 6954 1250 50  0001 C CNN
 F 2 "Inductor_SMD:L_0603_1608Metric" V 7030 1250 50  0001 C CNN
-F 3 "~" H 7100 1250 50  0001 C CNN
-F 4 "" H 7100 1250 50  0001 C CNN "Alt"
+F 3 "Ferrite_Bead_Small" H 7100 1250 50  0001 C CNN
+F 4 "Ferrite_Bead_Small" H 7100 1250 50  0001 C CNN "Alt"
 F 5 "490-5223-1-ND" H 7100 1250 50  0001 C CNN "Digikey"
-F 6 "470 Ohms @ 100MHz 1 Power Line Ferrite Bead 0603 1A 200mOhm" H 7100 1250 50  0001 C CNN "Error"
-F 7 "Ferrite_Bead_Small" H 7100 1250 50  0001 C CNN "LCSC"
+F 6 "Ferrite_Bead_Small" H 7100 1250 50  0001 C CNN "Error"
+F 7 "C97853" H 7100 1250 50  0001 C CNN "LCSC"
 F 8 "BLM18PG471SN1D" H 7100 1250 50  0001 C CNN "MPN"
-F 9 "~" H 7100 1250 50  0001 C CNN "Manufacturer"
-F 10 "" H 7100 1250 50  0001 C CNN "Mfr"
+F 9 "" H 7100 1250 50  0001 C CNN "Manufacturer"
+F 10 "470 Ohms @ 100MHz 1 Power Line Ferrite Bead 0603 1A 200mOhm" H 7100 1250 50  0001 C CNN "Mfr"
 F 11 "470 Ohms @ 100MHz 1 Power Line Ferrite Bead 0603 1A 200mOhm" H 7100 1250 50  0001 C CNN "Note"
-F 12 "490-5223-1-ND" H 7100 1250 50  0001 C CNN "Current"
-F 13 "BLM18PG471SN1D" H 7100 1250 50  0001 C CNN "Description"
+F 12 "Ferrite_Bead_Small" H 7100 1250 50  0001 C CNN "Current"
+F 13 "Ferrite_Bead_Small" H 7100 1250 50  0001 C CNN "Description"
 F 14 "81-BLM18PG471SN1D " H 7100 1250 50  0001 C CNN "Mouser"
 	1    7100 1250
@@
 F 0 "C141" H 8108 4296 50  0000 R CNN
 F 1 "4.7u" H 8108 4205 50  0000 R CNN
-F 2 "Capacitor_SMD:C_1206_3216Metric" H 8200 4250 50  0001 C CNN
+F 2 "Capacitor_SMD:C_0603_1608Metric" H 8200 4250 50  0001 C CNN
 F 3 "~" H 8200 4250 50  0001 C CNN
+F 4 "399-3482-1-ND" H 8200 4250 50  0001 C CNN "Digikey"
+F 5 "C86016" H 8200 4250 50  0001 C CNN "LCSC"
+F 6 "C0603C475K9PACTU" H 8200 4250 50  0001 C CNN "MPN"
+F 7 "CAP CER 4.7UF 6.3V X5R 0603" H 8200 4250 50  0001 C CNN "Note"
 	1    8200 4250
 	-1   0    0    -1

Commit message: 4layer layout WIP, 90%.
Changed SCD30 to reverse mount. 
Connected RGB led and button to io expander.
Connected all nets to micro.
Add jumper for CTS line.
Nettie GNDA and GND for W5500 Eth.
Changed EN_5V_BST to Global.
Bugfixes net names: LCD_CS
Parts:
- added NT201: Net-Tie_2, NetTie:NetTie-2_SMD_Pad0.5mm, symbol Device:Net-Tie_2
Connections:
- net GND: now also NT201.1
- net GNDA: now also NT201.2
Changed lines of the file:
@@
 Text HLabel 6150 2600 0    50   Input ~ 0
 ~ETH_RST
+$Comp
+L power:GND #PWR?
+U 1 1 6033D25D
+P 6350 4400
+AR Path="/6033D25D" Ref="#PWR?"  Part="1"
+AR Path="/5F9D72A5/6033D25D" Ref="#PWR?"  Part="1"
+AR Path="/5FCEDB09/6033D25D" Ref="#PWR0209"  Part="1"
+F 0 "#PWR0209" H 6350 4150 50  0001 C CNN
+F 1 "GND" H 6355 4227 50  0000 C CNN
+F 2 "" H 6350 4400 50  0001 C CNN
+F 3 "" H 6350 4400 50  0001 C CNN
+	1    6350 4400
+	-1   0    0    -1
+$EndComp
+$Comp
+L power:GNDA #PWR?
+U 1 1 6033D263
+P 6550 4400
+AR Path="/6033D263" Ref="#PWR?"  Part="1"
+AR Path="/5F9D72A5/6033D263" Ref="#PWR?"  Part="1"
+AR Path="/5FCEDB09/6033D263" Ref="#PWR0210"  Part="1"
+F 0 "#PWR0210" H 6550 4150 50  0001 C CNN
+F 1 "GNDA" H 6555 4227 50  0000 C CNN
+F 2 "" H 6550 4400 50  0001 C CNN
+F 3 "" H 6550 4400 50  0001 C CNN
+	1    6550 4400
+	1    0    0    -1
+$EndComp
+$Comp
+L Device:Net-Tie_2 NT201
+U 1 1 603434A7
+P 6450 4400
+F 0 "NT201" H 6450 4489 50  0000 C CNN
+F 1 "Net-Tie_2" H 6450 4490 50  0001 C CNN
+F 2 "NetTie:NetTie-2_SMD_Pad0.5mm" H 6450 4400 50  0001 C CNN
+F 3 "~" H 6450 4400 50  0001 C CNN
+	1    6450 4400
+	1    0    0    -1
+$EndComp
 $EndSCHEMATC

Commit message: Re-annotate all parts
Cleans up annotations
Parts:
- renumbered C110 to C201, C111 to C202, C112 to C203, C113 to C204, C114 to C205, C116 to C206, C117 to C207, C118 to C208, C119 to C209, C120 to C210, C121 to C211, C122 to C212, C123 to C213, C124 to C214, C125 to C215, C126 to C216, C127 to C217, C128 to C218, C129 to C219, FB101 to FB201, J101 to J201, JP103 to JP201, JP104 to JP202, JP105 to JP203, R116 to R201, R115 to R202, R114 to R203, R117 to R204, R118 to R205, R119 to R206, R121 to R207, R120 to R208, R125 to R209, R126 to R210, R127 to R211, R128 to R212, R129 to R213, R130 to R214, R131 to R215, R132 to R216, U105 to U201, Y101 to Y201

Commit message: Prefinal, layout done
Update FB to use inductor footprints
DNP net tie
Update diode symbol in power
Add battery voltage divider in power
Supply 5V power to aux sensor connector
Parts:
- NT201: DNP (none) -> 1
Changed lines of the file:
@@
 F 2 "NetTie:NetTie-2_SMD_Pad0.5mm" H 6450 4400 50  0001 C CNN
 F 3 "~" H 6450 4400 50  0001 C CNN
+F 4 "1" H 6450 4400 50  0001 C CNN "DNP"
 	1    6450 4400
 	1    0    0    -1

Commit message: BOM reduction and part picking
Parts:
- R201: Digikey (none) -> 311-10GRDKR-ND; LCSC (none) -> C109317; MPN (none) -> RC0603JR-0710RL; Note (none) -> RES SMD 10 OHM 5% 1/10W 0603
- R204, R205, R206: LCSC (none) -> C125933
- R209: LCSC (none) -> C105578
- R210, R211, R212, R213, R214, R215: LCSC (none) -> C98220
- R216: Digikey (none) -> 311-12.1KHRCT-ND; LCSC (none) -> C123417; MPN (none) -> RC0603FR-0712K1L; Note (none) -> RES SMD 12.1K OHM 1% 1/10W 0603
Changed lines of the file:
@@
 F 2 "Resistor_SMD:R_0603_1608Metric" H 2800 1400 60  0001 C CNN
 F 3 "" H 2800 1400 60  0001 C CNN
+F 4 "RC0603JR-0710RL" H 2800 1400 50  0001 C CNN "MPN"
+F 5 "311-10GRDKR-ND" H 2800 1400 50  0001 C CNN "Digikey"
+F 6 "RES SMD 10 OHM 5% 1/10W 0603" H 2800 1400 50  0001 C CNN "Note"
+F 7 " C109317 " H 2800 1400 50  0001 C CNN "LCSC"
 	1    2800 1400
 	1    0    0    1
@@
 F 5 "311-1.00KHRCT-ND" H 3800 1800 50  0001 C CNN "Digikey"
 F 6 "RES SMD 1K OHM 1% 1/10W 0603" H 3800 1800 50  0001 C CNN "Note"
+F 7 "C125933" H 3800 1800 50  0001 C CNN "LCSC"
 	1    3800 1800
 	0    1    -1   0
@@
 F 5 "311-1.00KHRCT-ND" H 3800 1600 50  0001 C CNN "Digikey"
 F 6 "RES SMD 1K OHM 1% 1/10W 0603" H 3800 1600 50  0001 C CNN "Note"
+F 7 "C125933" H 3800 1600 50  0001 C CNN "LCSC"
 	1    3800 1600
 	0    1    -1   0
@@
 F 5 "311-10.0KHRCT-ND" H 6250 4100 50  0001 C CNN "Digikey"
 F 6 "RES SMD 10K OHM 1% 1/10W 0603" H 6250 4100 50  0001 C CNN "Note"
+F 7 "C98220" H 6250 4100 50  0001 C CNN "LCSC"
 	1    6250 4100
 	0    -1   -1   0
@@
 F 5 "311-10.0KHRCT-ND" H 6250 3900 50  0001 C CNN "Digikey"
 F 6 "RES SMD 10K OHM 1% 1/10W 0603" H 6250 3900 50  0001 C CNN "Note"
+F 7 "C98220" H 6250 3900 50  0001 C CNN "LCSC"
 	1    6250 3900
 	0    -1   -1   0
@@
 F 5 "311-10.0KHRCT-ND" H 6250 3800 50  0001 C CNN "Digikey"
 F 6 "RES SMD 10K OHM 1% 1/10W 0603" H 6250 3800 50  0001 C CNN "Note"
+F 7 "C98220" H 6250 3800 50  0001 C CNN "LCSC"
 	1    6250 3800
 	0    -1   -1   0
@@
 F 5 "311-10.0KHRCT-ND" H 6250 3700 50  0001 C CNN "Digikey"
 F 6 "RES SMD 10K OHM 1% 1/10W 0603" H 6250 3700 50  0001 C CNN "Note"
+F 7 "C98220" H 6250 3700 50  0001 C CNN "LCSC"
 	1    6250 3700
 	0    -1   -1   0
@@
 F 5 "311-10.0KHRCT-ND" H 6250 3600 50  0001 C CNN "Digikey"
 F 6 "RES SMD 10K OHM 1% 1/10W 0603" H 6250 3600 50  0001 C CNN "Note"
+F 7 "C98220" H 6250 3600 50  0001 C CNN "LCSC"
 	1    6250 3600
 	0    -1   -1   0
@@
 F 5 "311-10.0KHRCT-ND" H 6250 3500 50  0001 C CNN "Digikey"
 F 6 "RES SMD 10K OHM 1% 1/10W 0603" H 6250 3500 50  0001 C CNN "Note"
+F 7 "C98220" H 6250 3500 50  0001 C CNN "LCSC"
 	1    6250 3500
 	0    -1   -1   0
@@
 F 5 "311-1.00KHRCT-ND" H 5850 2800 50  0001 C CNN "Digikey"
 F 6 "RES SMD 1K OHM 1% 1/10W 0603" H 5850 2800 50  0001 C CNN "Note"
+F 7 "C125933" H 5850 2800 50  0001 C CNN "LCSC"
 	1    5850 2800
 	0    -1   -1   0
@@
 F 5 "RC0603FR-071ML" H 5450 3300 50  0001 C CNN "MPN"
 F 6 "RES SMD 1M OHM 1% 1/10W 0603" H 5450 3300 50  0001 C CNN "Note"
+F 7 "C105578" H 5450 3300 50  0001 C CNN "LCSC"
 	1    5450 3300
 	0    1    1    0
@@
 F 2 "Resistor_SMD:R_0603_1608Metric" H 8600 4200 60  0001 C CNN
 F 3 "" H 8600 4200 60  0001 C CNN
+F 4 "RC0603FR-0712K1L" H 8600 4200 50  0001 C CNN "MPN"
+F 5 "311-12.1KHRCT-ND" H 8600 4200 50  0001 C CNN "Digikey"
+F 6 "RES SMD 12.1K OHM 1% 1/10W 0603" H 8600 4200 50  0001 C CNN "Note"
+F 7 "C123417" H 8600 4200 50  0001 C CNN "LCSC"
 	1    8600 4200
 	-1   0    0    1
