File: SD1.sch (KiCad schematic (older format))
At the start: 37 parts, among them J103 JST ZH 1.5mm 1x5, J107 FPC PMS, Q101 BSS138, Q102 PDTC114EU,115, SW103 Multidirection_Switch, SW104 Multifunction_Switch, U101 TLV70233_SOT23-5, U102 ER-TFTM028-4, U104 CC2652P, U106 EKMC1691111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

Commit message: Add BME280
Parts:
- added C? (x2): 0.1u, Capacitor_SMD:C_0603_1608Metric, symbol Device:C_Small
- added FB?: Ferrite_Bead_Small, Inductor_SMD:L_0603_1608Metric, symbol Device:Ferrite_Bead_Small
- added R? (x2): 10k, Resistor_SMD:R_0603_1608Metric, symbol Device:R_US
- added U?: BME280, Package_LGA:Bosch_LGA-8_2.5x2.5mm_P0.65mm_ClockwisePinNumbering, symbol Sensor:BME280
Connections:
- net +3V3: now also C?.1, FB?.2, R?.2, U?.6 (VDDIO)
- net GND: now also C?.2, C?.2, R?.2, U?.1 (GND), U?.7 (GND)
- net I2C_SCL: now also U?.4 (SCK)
- net I2C_SDA: now also U?.3 (SDI)
- new net: R?.1, U?.2 (CSB)
- new net: R?.1, U?.5 (SDO)
- new net: C?.1, FB?.1, U?.8 (VDD)
Other:
- note added: "I2C: 111011[0][rw]"
Changed lines of the file:
@@
 Text Notes 6250 8400 2    30   ~ 0
 Need to flip bc of cable
+Text Notes -35300 -1500 1    50   ~ 0
+SERCOM 0
+Text Notes -35300 -1500 1    50   ~ 0
+SERCOM 0
+Text Notes -35300 -1500 1    50   ~ 0
+SERCOM 0
+Text Notes -35300 -1500 1    50   ~ 0
+SERCOM 0
+$Comp
+L power:GND #PWR?
+U 1 1 5FB0CAA2
+P 12050 8800
+F 0 "#PWR?" H 12050 8550 50  0001 C CNN
+F 1 "GND" H 12055 8627 50  0000 C CNN
+F 2 "" H 12050 8800 50  0001 C CNN
+F 3 "" H 12050 8800 50  0001 C CNN
+	1    12050 8800
+	1    0    0    -1
+$EndComp
+Wire Wire Line
+	11500 7150 11500 7100
+$Comp
+L power:+3.3V #PWR?
+U 1 1 5FB0CAA9
+P 11500 7050
+F 0 "#PWR?" H 11500 6900 50  0001 C CNN
+F 1 "+3.3V" H 11515 7223 50  0000 C CNN
+F 2 "" H 11500 7050 50  0001 C CNN
+F 3 "" H 11500 7050 50  0001 C CNN
+	1    11500 7050
+	1    0    0    -1
+$EndComp
+$Comp
+L Sensor:BME280 U?
+U 1 1 5FB0CAB4
+P 11950 8100
+F 0 "U?" H 11521 8146 50  0000 R CNN
+F 1 "BME280" H 11521 8055 50  0000 R CNN
+F 2 "Package_LGA:Bosch_LGA-8_2.5x2.5mm_P0.65mm_ClockwisePinNumbering" H 13450 7650 50  0001 C CNN
+F 3 "https://www.bosch-sensortec.com/media/boschsensortec/downloads/datasheets/bst-bme280-ds002.pdf" H 11950 7900 50  0001 C CNN
+F 4 "BME280" H 11950 8100 50  0001 C CNN "MPN"
+F 5 "828-1063-1-ND" H 11950 8100 50  0001 C CNN "Digikey"
+F 6 "Humidity Temperature Sensor 0 ~ 100% RH I²C, SPI ±3% 1s Surface Mount" H 11950 8100 50  0001 C CNN "Note"
+F 7 "262-BME280" H 11950 8100 50  0001 C CNN "Mouser"
+F 8 " C92489 " H 11950 8100 50  0001 C CNN "LCSC"
+	1    11950 8100
+	1    0    0    -1
+$EndComp
+Wire Wire Line
+	12550 8400 12650 8400
+$Comp
+L power:+3.3V #PWR?
+U 1 1 5FB0CABB
+P 13050 8350
+F 0 "#PWR?" H 13050 8200 50  0001 C CNN
+F 1 "+3.3V" H 13065 8523 50  0000 C CNN
+F 2 "" H 13050 8350 50  0001 C CNN
+F 3 "" H 13050 8350 50  0001 C CNN
+	1    13050 8350
+	1    0    0    -1
+$EndComp
+Wire Wire Line
+	13050 8400 13050 8350
+$Comp
+L Device:R_US R?
+U 1 1 5FB0CAC7
+P 12800 7800
+F 0 "R?" V 13005 7800 50  0000 C CNN
+F 1 "10k" V 12914 7800 50  0000 C CNN
+F 2 "Resistor_SMD:R_0603_1608Metric" H 12800 7800 60  0001 C CNN
+F 3 "" H 12800 7800 60  0001 C CNN
+F 4 "RC0603FR-0710KL" H 12800 7800 50  0001 C CNN "MPN"
+F 5 "311-10.0KHRCT-ND" H 12800 7800 50  0001 C CNN "Digikey"
+F 6 "RES SMD 10K OHM 1% 1/10W 0603" H 12800 7800 50  0001 C CNN "Note"
+	1    12800 7800
+	0    -1   -1   0
+$EndComp
+$Comp
+L Device:R_US R?
+U 1 1 5FB0CAD0
+P 12800 8400
+F 0 "R?" V 12687 8400 50  0000 C CNN
+F 1 "10k" V 12596 8400 50  0000 C CNN
+F 2 "Resistor_SMD:R_0603_1608Metric" H 12800 8400 60  0001 C CNN
+F 3 "" H 12800 8400 60  0001 C CNN
+F 4 "RC0603FR-0710KL" H 12800 8400 50  0001 C CNN "MPN"
+F 5 "311-10.0KHRCT-ND" H 12800 8400 50  0001 C CNN "Digikey"
+F 6 "RES SMD 10K OHM 1% 1/10W 0603" H 12800 8400 50  0001 C CNN "Note"
+	1    12800 8400
+	0    -1   -1   0
+$EndComp
+$Comp
+L Device:Ferrite_Bead_Small FB?
+U 1 1 5FB0CADA
+P 11950 7100
+F 0 "FB?" V 11805 7100 50  0000 C CNN
+F 1 "Ferrite_Bead_Small" V 11804 7100 50  0001 C CNN
+F 2 "Inductor_SMD:L_0603_1608Metric" V 11880 7100 50  0001 C CNN
+F 3 "~" H 11950 7100 50  0001 C CNN
+F 4 "BLM18PG471SN1D" H 11950 7100 50  0001 C CNN "MPN"
+F 5 "81-BLM18PG471SN1D " H 11950 7100 50  0001 C CNN "Mouser"
+F 6 "490-5223-1-ND" H 11950 7100 50  0001 C CNN "Digikey"
+F 7 "470 Ohms @ 100MHz 1 Power Line Ferrite Bead 0603 1A 200mOhm" H 11950 7100 50  0001 C CNN "Note"
+	1    11950 7100
+	0    1    1    0
+$EndComp
+Wire Wire Line
+	11850 7100 11500 7100
+Wire Wire Line
+	11500 7050 11500 7100
+Connection ~ 11500 7100
+$Comp
+L power:GND #PWR?
+U 1 1 5FB0CAE3
+P 12300 7400
+F 0 "#PWR?" H 12300 7150 50  0001 C CNN
+F 1 "GND" H 12305 7227 50  0000 C CNN
+F 2 "" H 12300 7400 50  0001 C CNN
+F 3 "" H 12300 7400 50  0001 C CNN
+	1    12300 7400
+	1    0    0    -1
+$EndComp
+Connection ~ 12050 7100
+Wire Wire Line
+	12050 7100 12300 7100
+Wire Wire Line
+	12300 7150 12300 7100
+Wire Wire Line
+	12300 7350 12300 7400
+$Comp
+L power:GND #PWR?
+U 1 1 5FB0CAED
+P 11500 7400
+F 0 "#PWR?" H 11500 7150 50  0001 C CNN
+F 1 "GND" H 11505 7227 50  0000 C CNN
+F 2 "" H 11500 7400 50  0001 C CNN
+F 3 "" H 11500 7400 50  0001 C CNN
+	1    11500 7400
+	1    0    0    -1
+$EndComp
+Wire Wire Line
+	11500 7400 11500 7350
+Wire Wire Line
+	11850 7100 11850 7500
+Connection ~ 11850 7100
+Wire Wire Line
+	12050 7100 12050 7500
+$Comp
+L Device:C_Small C?
+U 1 1 5FB0CAFA
+P 11500 7250
+AR Path="/5E360A9B/5FB0CAFA" Ref="C?"  Part="1"
+AR Path="/5FB0CAFA" Ref="C?"  Part="1"
+AR Path="/5E49A000/5FB0CAFA" Ref="C?"  Part="1"
+AR Path="/5E5C8043/5E49A000/5FB0CAFA" Ref="C?"  Part="1"
+AR Path="/5E5C8043/5EAB3002/5FB0CAFA" Ref="C?"  Part="1"
+AR Path="/5E5C8043/5FB0CAFA" Ref="C?"  Part="1"
+F 0 "C?" H 11592 7296 50  0000 L CNN
+F 1 "0.1u" H 11592 7205 50  0000 L CNN
+F 2 "Capacitor_SMD:C_0603_1608Metric" H 11500 7250 50  0001 C CNN
+F 3 "~" H 11500 7250 50  0001 C CNN
+F 4 "0603B104K500CT" H 11500 7250 50  0001 C CNN "MPN"
+F 5 "1292-1643-1-ND" H 11500 7250 50  0001 C CNN "Digikey"
+F 6 "CAP CER 0.1UF 50V X7R 0603" H 11500 7250 50  0001 C CNN "Note"
+	1    11500 7250
+	1    0    0    -1
+$EndComp
+$Comp
+L Device:C_Small C?
+U 1 1 5FB0CB03
+P 12300 7250
+AR Path="/5E360A9B/5FB0CB03" Ref="C?"  Part="1"
+AR Path="/5FB0CB03" Ref="C?"  Part="1"
+AR Path="/5E49A000/5FB0CB03" Ref="C?"  Part="1"
+AR Path="/5E5C8043/5E49A000/5FB0CB03" Ref="C?"  Part="1"
+AR Path="/5E5C8043/5EAB3002/5FB0CB03" Ref="C?"  Part="1"
+AR Path="/5E5C8043/5FB0CB03" Ref="C?"  Part="1"
+F 0 "C?" H 12392 7296 50  0000 L CNN
+F 1 "0.1u" H 12392 7205 50  0000 L CNN
+F 2 "Capacitor_SMD:C_0603_1608Metric" H 12300 7250 50  0001 C CNN
+F 3 "~" H 12300 7250 50  0001 C CNN
+F 4 "0603B104K500CT" H 12300 7250 50  0001 C CNN "MPN"
+F 5 "1292-1643-1-ND" H 12300 7250 50  0001 C CNN "Digikey"
+F 6 "CAP CER 0.1UF 50V X7R 0603" H 12300 7250 50  0001 C CNN "Note"
+	1    12300 7250
+	1    0    0    -1
+$EndComp
+Wire Wire Line
+	12550 7800 12650 7800
+$Comp
+L power:GND #PWR?
+U 1 1 5FB0CB0B
+P 13050 7850
+F 0 "#PWR?" H 13050 7600 50  0001 C CNN
+F 1 "GND" H 13055 7677 50  0000 C CNN
+F 2 "" H 13050 7850 50  0001 C CNN
+F 3 "" H 13050 7850 50  0001 C CNN
+	1    13050 7850
+	1    0    0    -1
+$EndComp
+Wire Wire Line
+	12950 7800 13050 7800
+Wire Wire Line
+	13050 7800 13050 7850
+Wire Wire Line
+	12950 8400 13050 8400
+Text GLabel 12550 8200 2    40   BiDi ~ 0
+I2C_SDA
+Text GLabel 12550 8000 2    40   Input ~ 0
+I2C_SCL
+Wire Wire Line
+	12050 8700 12050 8750
+Wire Wire Line
+	12050 8750 11850 8750
+Wire Wire Line
+	11850 8750 11850 8700
+Connection ~ 12050 8750
+Wire Wire Line
+	12050 8750 12050 8800
+Text Notes 12600 8600 2    30   ~ 0
+I2C: 111011[0][rw]
 $EndSCHEMATC
