File: poe.sch (KiCad schematic (older format))
At the start: 70 parts, among them J301 PJ-102AH, J302 PJ-102AH, J303 Conn_01x02, J304 Conn_01x02, Q301 DMMT5401, Q302 DMMT5401, Q303 FDT86244, T301 HR051067, U301 TPS23753A, U302 TL431A, U303 TCMT1107

Commit message: BOM reduction and part picking
Parts:
- added R326: 1k, Resistor_SMD:R_0603_1608Metric, symbol Device:R_US
- C317: footprint Capacitor_SMD:C_0805_2012Metric -> Capacitor_SMD:C_0603_1608Metric; Digikey 1276-1066-1-ND -> 587-2984-1-ND; Error 10% -> (none); LCSC C116352 -> (none); MPN CL21B105KAFNNNE -> TMK107B7105KA-T; Note CAP CER 1UF X7R 16V 0805 -> CAP CER 1UF 25V X7R 0603; Size 0805 -> (none); Type X7R -> (none); Voltage 16V -> (none)
- Q301: value DMMT5401 -> DMP3098L-7
- R302: value 20 -> 22.1; footprint Resistor_SMD:R_0805_2012Metric -> Resistor_SMD:R_0603_1608Metric; Digikey 311-20ARCT-ND -> 311-22.1HRCT-ND; Error 5% -> (none); LCSC C137459 -> C137767; MPN RC0805JR-0720RL -> RC0603FR-0722R1L; Note RES SMD 20 OHM 5% 1/10W 0805 -> RES SMD 22.1 OHM 1% 1/10W 0603; Power 1/10W -> (none); Size 0805 -> (none)
- R309: LCSC (none) -> C98220
- R310: Digikey (none) -> 311-47.5KHRCT-ND; LCSC (none) -> C137715; MPN (none) -> RC0603FR-0747K5L; Note (none) -> RES SMD 47.5K OHM 1% 1/10W 0603
- R312: LCSC (none) -> C421678, C20464
- R313, R322: LCSC (none) -> C125933
- R314: Digikey (none) -> 311-10.0KHRCT-ND; LCSC (none) -> C98220; MPN (none) -> RC0603FR-0710KL; Note (none) -> RES SMD 10K OHM 1% 1/10W 0603
- R323: value 2k -> 1k; Digikey YAG3590CT-ND -> 311-1.00KHRCT-ND; MPN AC0603FR-072KL -> RC0603FR-071KL; Note RES SMD 2K OHM 1% 1/16W 0603 -> RES SMD 1K OHM 1% 1/10W 0603
Connections:
- net at C315.1, R320.1, U301.2 (VB): now also R326.1; no longer R323.1
- new net: R323.1, R326.2
Changed lines of the file:
@@
 AR Path="/5FCEDB09/5FAC6B33/5F89CD2C" Ref="R323"  Part="1"
 F 0 "R323" H 8518 7346 50  0000 L CNN
-F 1 "2k" H 8518 7255 50  0000 L CNN
+F 1 "1k" H 8518 7255 50  0000 L CNN
 F 2 "Resistor_SMD:R_0603_1608Metric" H 8450 7300 50  0001 C CNN
 F 3 "~" H 8450 7300 50  0001 C CNN
@@
 F 5 "1%" H 8450 7300 50  0001 C CNN "Error"
 F 6 "0603" H 8450 7300 50  0001 C CNN "Size"
-F 7 "RES SMD 2K OHM 1% 1/16W 0603" H 8450 7300 50  0001 C CNN "Note"
-F 8 "YAG3590CT-ND" H 8450 7300 50  0001 C CNN "Digikey"
+F 7 "RES SMD 1K OHM 1% 1/10W 0603" H 8450 7300 50  0001 C CNN "Note"
+F 8 "311-1.00KHRCT-ND" H 8450 7300 50  0001 C CNN "Digikey"
 F 9 "C125933" H 8450 7300 50  0001 C CNN "LCSC"
-F 10 "AC0603FR-072KL" H 8450 7300 50  0001 C CNN "MPN"
+F 10 "RC0603FR-071KL" H 8450 7300 50  0001 C CNN "MPN"
 	1    8450 7300
 	1    0    0    -1
@@
 F 0 "C317" H 11042 6996 50  0000 L CNN
 F 1 "1u" H 11042 6905 50  0000 L CNN
-F 2 "Capacitor_SMD:C_0805_2012Metric" H 10950 6950 50  0001 C CNN
+F 2 "Capacitor_SMD:C_0603_1608Metric" H 10950 6950 50  0001 C CNN
 F 3 "~" H 10950 6950 50  0001 C CNN
-F 4 "16V" H 10950 6950 50  0001 C CNN "Voltage"
-F 5 "10%" H 10950 6950 50  0001 C CNN "Error"
-F 6 "X7R" H 10950 6950 50  0001 C CNN "Type"
-F 7 "0805" H 10950 6950 50  0001 C CNN "Size"
-F 8 "1276-1066-1-ND" H 10950 6950 50  0001 C CNN "Digikey"
-F 9 "C116352" H 10950 6950 50  0001 C CNN "LCSC"
-F 10 "CL21B105KAFNNNE" H 10950 6950 50  0001 C CNN "MPN"
-F 11 "CAP CER 1UF X7R 16V 0805" H 10950 6950 50  0001 C CNN "Note"
+F 4 "" H 10950 6950 50  0001 C CNN "Voltage"
+F 5 "" H 10950 6950 50  0001 C CNN "Error"
+F 6 "" H 10950 6950 50  0001 C CNN "Type"
+F 7 "" H 10950 6950 50  0001 C CNN "Size"
+F 8 "587-2984-1-ND" H 10950 6950 50  0001 C CNN "Digikey"
+F 9 "TMK107B7105KA-T" H 10950 6950 50  0001 C CNN "MPN"
+F 10 "CAP CER 1UF 25V X7R 0603" H 10950 6950 50  0001 C CNN "Note"
 	1    10950 6950
 	1    0    0    -1
@@
 $EndComp
 $Comp
-L Device:R_US R?
-U 1 1 5F976A36
-P 11000 4600
-AR Path="/5F81C554/5F976A36" Ref="R?"  Part="1"
-AR Path="/5F9D72A5/5FA9FFA2/5F976A36" Ref="R?"  Part="1"
-AR Path="/5FAC6B33/5F976A36" Ref="R?"  Part="1"
-AR Path="/5FCEDB09/5FAC6B33/5F976A36" Ref="R302"  Part="1"
-F 0 "R302" V 10795 4600 50  0000 C CNN
-F 1 "20" V 10886 4600 50  0000 C CNN
-F 2 "Resistor_SMD:R_0805_2012Metric" H 11000 4600 50  0001 C CNN
-F 3 "~" H 11000 4600 50  0001 C CNN
-F 4 "1/10W" V 11000 4600 50  0001 C CNN "Power"
-F 5 "5%" V 11000 4600 50  0001 C CNN "Error"
-F 6 "0805" V 11000 4600 50  0001 C CNN "Size"
-F 7 "RES SMD 20 OHM 5% 1/10W 0805" H 11000 4600 50  0001 C CNN "Note"
-F 8 "311-20ARCT-ND" H 11000 4600 50  0001 C CNN "Digikey"
-F 9 "C137459" H 11000 4600 50  0001 C CNN "LCSC"
-F 10 "RC0805JR-0720RL" H 11000 4600 50  0001 C CNN "MPN"
-	1    11000 4600
-	0    1    1    0
-$EndComp
-$Comp
 L Device:C_Small C?
 U 1 1 5F977204
@@
 F 5 "1%" H 10950 6200 50  0001 C CNN "Error"
 F 6 "0603" H 10950 6200 50  0001 C CNN "Size"
+F 7 "311-10.0KHRCT-ND" H 10950 6200 50  0001 C CNN "Digikey"
+F 8 "C98220" H 10950 6200 50  0001 C CNN "LCSC"
+F 9 "RC0603FR-0710KL" H 10950 6200 50  0001 C CNN "MPN"
+F 10 "RES SMD 10K OHM 1% 1/10W 0603" H 10950 6200 50  0001 C CNN "Note"
 	1    10950 6200
 	1    0    0    -1
@@
 F 7 "RES SMD 1K OHM 1% 1/10W 0603" H 13500 7050 50  0001 C CNN "Note"
 F 8 "311-1.00KHRCT-ND" H 13500 7050 50  0001 C CNN "Digikey"
-F 9 "" H 13500 7050 50  0001 C CNN "LCSC"
+F 9 "C125933" H 13500 7050 50  0001 C CNN "LCSC"
 F 10 "RC0603FR-071KL" H 13500 7050 50  0001 C CNN "MPN"
 	1    13500 7050
@@
 	8950 5850 9000 5850
 Wire Wire Line
-	8450 7150 8450 6450
+	8450 7150 8450 7100
 Wire Wire Line
 	11150 4600 11250 4600
@@
 F 6 "2010" H 9850 5900 50  0001 C CNN "Size"
 F 7 "RES SMD 82 OHM 5% 1/2W 2010" H 9850 5900 50  0001 C CNN "Note"
+F 8 "C421678, C20464" H 9850 5900 50  0001 C CNN "LCSC"
 	1    9850 5900
 	1    0    0    -1
@@
 F 8 "RC0603FR-071KL" H 10700 6200 50  0001 C CNN "MPN"
 F 9 "RES SMD 1K OHM 1% 1/10W 0603" H 10700 6200 50  0001 C CNN "Note"
+F 10 "C125933" H 10700 6200 50  0001 C CNN "LCSC"
 	1    10700 6200
 	1    0    0    -1
@@
 AR Path="/5FCEDB09/5FAC6B33/5FEFAC35" Ref="Q301"  Part="1"
 F 0 "Q301" V 14342 5050 50  0000 C CNN
-F 1 "DMMT5401" V 14251 5050 50  0000 C CNN
+F 1 "DMP3098L-7" V 14251 5050 50  0000 C CNN
 F 2 "Package_TO_SOT_SMD:SOT-23-6" H 14200 5150 50  0001 C CNN
 F 3 "~" H 14000 5050 50  0001 C CNN
@@
 F 5 "311-10.0KHRCT-ND" H 13550 5750 50  0001 C CNN "Digikey"
 F 6 "RES SMD 10K OHM 1% 1/10W 0603" H 13550 5750 50  0001 C CNN "Note"
+F 7 "C98220" H 13550 5750 50  0001 C CNN "LCSC"
 	1    13550 5750
 	1    0    0    -1
@@
 F 2 "Resistor_SMD:R_0603_1608Metric" H 14450 5750 60  0001 C CNN
 F 3 "" H 14450 5750 60  0001 C CNN
+F 4 "311-47.5KHRCT-ND" H 14450 5750 50  0001 C CNN "Digikey"
+F 5 " C137715 " H 14450 5750 50  0001 C CNN "LCSC"
+F 6 "RC0603FR-0747K5L" H 14450 5750 50  0001 C CNN "MPN"
+F 7 "RES SMD 47.5K OHM 1% 1/10W 0603" H 14450 5750 50  0001 C CNN "Note"
 	1    14450 5750
 	-1   0    0    1
@@
 Wire Wire Line
 	2600 4450 2050 4450
+$Comp
+L Device:R_US R?
+U 1 1 5FE7760F
+P 11000 4600
+AR Path="/5FED2126/5FE7760F" Ref="R?"  Part="1"
+AR Path="/5FCEDB09/5FAC6B33/5FE7760F" Ref="R302"  Part="1"
+F 0 "R302" V 10795 4600 50  0000 C CNN
+F 1 "22.1" V 10886 4600 50  0000 C CNN
+F 2 "Resistor_SMD:R_0603_1608Metric" H 11000 4600 60  0001 C CNN
+F 3 "" H 11000 4600 60  0001 C CNN
+F 4 "311-22.1HRCT-ND" H 11000 4600 50  0001 C CNN "Digikey"
+F 5 "C137767 " H 11000 4600 50  0001 C CNN "LCSC"
+F 6 "RC0603FR-0722R1L" H 11000 4600 50  0001 C CNN "MPN"
+F 7 "RES SMD 22.1 OHM 1% 1/10W 0603" H 11000 4600 50  0001 C CNN "Note"
+	1    11000 4600
+	0    1    1    0
+$EndComp
+$Comp
+L Device:R_US R?
+U 1 1 5FE94C99
+P 8450 6950
+AR Path="/5F81C554/5FE94C99" Ref="R?"  Part="1"
+AR Path="/5F9D72A5/5FA9FFA2/5FE94C99" Ref="R?"  Part="1"
+AR Path="/5FAC6B33/5FE94C99" Ref="R?"  Part="1"
+AR Path="/5FCEDB09/5FAC6B33/5FE94C99" Ref="R326"  Part="1"
+F 0 "R326" H 8518 6996 50  0000 L CNN
+F 1 "1k" H 8518 6905 50  0000 L CNN
+F 2 "Resistor_SMD:R_0603_1608Metric" H 8450 6950 50  0001 C CNN
+F 3 "~" H 8450 6950 50  0001 C CNN
+F 4 "1/16W" H 8450 6950 50  0001 C CNN "Power"
+F 5 "" H 8450 6950 50  0001 C CNN "Error"
+F 6 "0603" H 8450 6950 50  0001 C CNN "Size"
+F 7 "311-1.00KHRCT-ND" H 8450 6950 50  0001 C CNN "Digikey"
+F 8 "RC0603FR-071KL" H 8450 6950 50  0001 C CNN "MPN"
+F 9 "RES SMD 1K OHM 1% 1/10W 0603" H 8450 6950 50  0001 C CNN "Note"
+F 10 "C125933" H 8450 6950 50  0001 C CNN "LCSC"
+	1    8450 6950
+	1    0    0    -1
+$EndComp
+Wire Wire Line
+	8450 6800 8450 6450
 $EndSCHEMATC

Commit message: Prep for gerber export
Update fields
Align standoff holes
Parts:
- R318: Digikey (none) -> 273-KDV12FR560ETCT-ND; LCSC (none) -> C175807; MPN (none) -> KDV12FR560ET; Note RES SMD 0.56 OHM 1% 1/4W 1206 -> RES 560M OHM 1% 1/2W 1206
Changed lines of the file:
@@
 F 5 "1%" H 9300 6600 50  0001 C CNN "Error"
 F 6 "1206" H 9300 6600 50  0001 C CNN "Size"
-F 7 "RES SMD 0.56 OHM 1% 1/4W 1206" H 9300 6600 50  0001 C CNN "Note"
+F 7 "RES 560M OHM 1% 1/2W 1206" H 9300 6600 50  0001 C CNN "Note"
+F 8 "KDV12FR560ET" H 9300 6600 50  0001 C CNN "MPN"
+F 9 "273-KDV12FR560ETCT-ND" H 9300 6600 50  0001 C CNN "Digikey"
+F 10 "C175807" H 9300 6600 50  0001 C CNN "LCSC"
 	1    9300 6600
 	1    0    0    -1
