File: poe.sch (KiCad schematic (older format))
At the start: 71 parts, among them J301 PJ-102AH, J302 PJ-102AH, J303 Conn_01x02, J304 Conn_01x02, Q301 DMP3098L-7, Q302 DMMT5401, Q303 FDT86244, T301 HR051067, U301 TPS23753A, U302 TL431A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

Commit message: Schematic field cleanup
Remove stray spaces
Cleaned up duplicate fields
Normalize: 100pF (C314 C803 C807) and 47uF  (C308 C310 C804 C805) according to r0 order
Parts:
- C305: value 680pF -> 680p
- C308, C310: value 47uF -> 47u; Digikey (none) -> 587-5922-1-ND
- C309: value 47uF -> 47u
- C314: value 100pF -> 100p
- C316: value 8.2nF -> 8.2n
- FB301, FB302: Manufacturer Chilisin Elec -> Chilisin Elec; Note 11Ω @ 100MHz 4A 1 20mΩ 0603 Ferrite Beads -> 11Ω @ 100MHz 4A 1 20mΩ 0603 Ferrite Beads
- L301: Note 4.7uH ±20% 2A 60mΩ SMD,4x4x3mm -> 4.7uH ±20% 2A 60mΩ SMD,4x4x3mm
- R302: LCSC C137767 -> C137767
- R310: LCSC C137715 -> C137715
Changed lines of the file:
@@
 F 5 "C280672" H 4500 4250 50  0001 C CNN "LCSC"
 F 6 "PBY160808T-110Y-N" H 4500 4250 50  0001 C CNN "MPN"
-F 7 " Chilisin Elec" H 4500 4250 50  0001 C CNN "Manufacturer"
-F 8 " 11Ω @ 100MHz 4A 1 20mΩ 0603 Ferrite Beads" H 4500 4250 50  0001 C CNN "Note"
+F 7 "Chilisin Elec" H 4500 4250 50  0001 C CNN "Manufacturer"
+F 8 "11Ω @ 100MHz 4A 1 20mΩ 0603 Ferrite Beads" H 4500 4250 50  0001 C CNN "Note"
 	1    4500 4250
 	0    1    1    0
@@
 F 5 "C280672" H 4500 6950 50  0001 C CNN "LCSC"
 F 6 "PBY160808T-110Y-N" H 4500 6950 50  0001 C CNN "MPN"
-F 7 " Chilisin Elec" H 4500 6950 50  0001 C CNN "Manufacturer"
-F 8 " 11Ω @ 100MHz 4A 1 20mΩ 0603 Ferrite Beads" H 4500 6950 50  0001 C CNN "Note"
+F 7 "Chilisin Elec" H 4500 6950 50  0001 C CNN "Manufacturer"
+F 8 "11Ω @ 100MHz 4A 1 20mΩ 0603 Ferrite Beads" H 4500 6950 50  0001 C CNN "Note"
 	1    4500 6950
 	0    1    1    0
@@
 F 5 "C206284, C326301, C15269" H 7700 4250 50  0001 C CNN "LCSC"
 F 6 "SLW4030S4R7MST" H 7700 4250 50  0001 C CNN "MPN"
-F 7 "4.7uH ±20% 2A 60mΩ SMD,4x4x3mm " H 7700 4250 50  0001 C CNN "Note"
+F 7 "4.7uH ±20% 2A 60mΩ SMD,4x4x3mm" H 7700 4250 50  0001 C CNN "Note"
 	1    7700 4250
 	0    -1   -1   0
@@
 AR Path="/5FCEDB09/5FAC6B33/5F8F91D7" Ref="C316"  Part="1"
 F 0 "C316" V 12271 6850 50  0000 C CNN
-F 1 "8.2nF" V 12362 6850 50  0000 C CNN
+F 1 "8.2n" V 12362 6850 50  0000 C CNN
 F 2 "Capacitor_SMD:C_0603_1608Metric" H 12500 6850 50  0001 C CNN
 F 3 "~" H 12500 6850 50  0001 C CNN
@@
 AR Path="/5FCEDB09/5FAC6B33/5F91C906" Ref="C314"  Part="1"
 F 0 "C314" V 12121 6450 50  0000 C CNN
-F 1 "100pF" V 12212 6450 50  0000 C CNN
+F 1 "100p" V 12212 6450 50  0000 C CNN
 F 2 "Capacitor_SMD:C_0603_1608Metric" H 12350 6450 50  0001 C CNN
 F 3 "~" H 12350 6450 50  0001 C CNN
@@
 AR Path="/5FCEDB09/5FAC6B33/5F977204" Ref="C305"  Part="1"
 F 0 "C305" V 11121 4600 50  0000 C CNN
-F 1 "680pF" V 11212 4600 50  0000 C CNN
+F 1 "680p" V 11212 4600 50  0000 C CNN
 F 2 "Capacitor_SMD:C_0603_1608Metric" H 11350 4600 50  0001 C CNN
 F 3 "~" H 11350 4600 50  0001 C CNN
@@
 AR Path="/5FCEDB09/5FAC6B33/5FD7B52B" Ref="C308"  Part="1"
 F 0 "C308" H 11659 5246 50  0000 R CNN
-F 1 "47uF" H 11659 5155 50  0000 R CNN
+F 1 "47u" H 11659 5155 50  0000 R CNN
 F 2 "Capacitor_SMD:C_1210_3225Metric" H 11750 5200 50  0001 C CNN
 F 3 "" H 11750 5200 50  0001 C CNN
@@
 F 9 "1210X476K160CT" H 11750 5200 50  0001 C CNN "MPN"
 F 10 "CAP CER 47UF X5R 10V 1210" H 11750 5200 50  0001 C CNN "Note"
+F 11 "587-5922-1-ND" H 11750 5200 50  0001 C CNN "Digikey"
 	1    11750 5200
 	1    0    0    -1
@@
 AR Path="/5FCEDB09/5FAC6B33/5FD7B535" Ref="C309"  Part="1"
 F 0 "C309" H 12141 5246 50  0000 L CNN
-F 1 "47uF" H 12141 5155 50  0000 L CNN
+F 1 "47u" H 12141 5155 50  0000 L CNN
 F 2 "Capacitor_SMD:CP_Elec_4x5.8" H 12050 5200 50  0001 C CNN
 F 3 "~" H 12050 5200 50  0001 C CNN
@@
 AR Path="/5FCEDB09/5FAC6B33/5FD7B53F" Ref="C310"  Part="1"
 F 0 "C310" H 12542 5246 50  0000 L CNN
-F 1 "47uF" H 12542 5155 50  0000 L CNN
+F 1 "47u" H 12542 5155 50  0000 L CNN
 F 2 "Capacitor_SMD:C_1210_3225Metric" H 12450 5200 50  0001 C CNN
 F 3 "~" H 12450 5200 50  0001 C CNN
@@
 F 9 "1210X476K160CT" H 12450 5200 50  0001 C CNN "MPN"
 F 10 "CAP CER 47UF X5R 10V 1210" H 12450 5200 50  0001 C CNN "Note"
+F 11 "587-5922-1-ND" H 12450 5200 50  0001 C CNN "Digikey"
 	1    12450 5200
 	1    0    0    -1
@@
 F 3 "" H 14450 5750 60  0001 C CNN
 F 4 "311-47.5KHRCT-ND" H 14450 5750 50  0001 C CNN "Digikey"
-F 5 " C137715 " H 14450 5750 50  0001 C CNN "LCSC"
+F 5 "C137715" H 14450 5750 50  0001 C CNN "LCSC"
 F 6 "RC0603FR-0747K5L" H 14450 5750 50  0001 C CNN "MPN"
 F 7 "RES SMD 47.5K OHM 1% 1/10W 0603" H 14450 5750 50  0001 C CNN "Note"
@@
 F 3 "" H 11000 4600 60  0001 C CNN
 F 4 "311-22.1HRCT-ND" H 11000 4600 50  0001 C CNN "Digikey"
-F 5 "C137767 " H 11000 4600 50  0001 C CNN "LCSC"
+F 5 "C137767" H 11000 4600 50  0001 C CNN "LCSC"
 F 6 "RC0603FR-0722R1L" H 11000 4600 50  0001 C CNN "MPN"
 F 7 "RES SMD 22.1 OHM 1% 1/10W 0603" H 11000 4600 50  0001 C CNN "Note"
