File: sensor_voc.sch (KiCad schematic (older format))
At the start: 5 parts, among them U601 CCS811

Commit message: Continue part picking
Parts:
- C601: value 100nF -> 0.1u; Digikey (none) -> 1292-1643-1-ND; MPN (none) -> 0603B104K500CT; Note (none) -> CAP CER 0.1UF 50V X7R 0603
Changed lines of the file:
@@
 P 6500 3350
 F 0 "C601" H 6408 3396 50  0000 R CNN
-F 1 "100nF" H 6408 3305 50  0000 R CNN
+F 1 "0.1u" H 6408 3305 50  0000 R CNN
 F 2 "Capacitor_SMD:C_0603_1608Metric" H 6500 3350 50  0001 C CNN
 F 3 "" H 6500 3350 50  0001 C CNN
+F 4 "1292-1643-1-ND" H 6500 3350 50  0001 C CNN "Digikey"
+F 5 "0603B104K500CT" H 6500 3350 50  0001 C CNN "MPN"
+F 6 "CAP CER 0.1UF 50V X7R 0603" H 6500 3350 50  0001 C CNN "Note"
 	1    6500 3350
 	-1   0    0    -1

Commit message: Re-annotate all parts
Cleans up annotations
Parts:
- renumbered C601 to C501, R601 to R501, R602 to R502, R603 to R503, U601 to U501
Changed lines of the file:
@@
 	5200 3200 5200 3150
 $Comp
-L Device:R_US R602
+L Device:R_US R502
 U 1 1 5E9445B2
 P 5200 3350
-F 0 "R602" V 5280 3350 50  0000 C CNN
+F 0 "R502" V 5280 3350 50  0000 C CNN
 F 1 "10k" V 5120 3350 50  0000 C CNN
 F 2 "Resistor_SMD:R_0603_1608Metric" H 5200 3350 60  0001 C CNN
@@
 	4850 4600 4850 4550
 $Comp
-L power:GND #PWR0602
+L power:GND #PWR0502
 U 1 1 5E897F37
 P 5700 4650
-F 0 "#PWR0602" H 5700 4400 50  0001 C CNN
+F 0 "#PWR0502" H 5700 4400 50  0001 C CNN
 F 1 "GND" H 5705 4477 50  0000 C CNN
 F 2 "" H 5700 4650 50  0001 C CNN
@@
 	5300 4100 4850 4100
 $Comp
-L Device:R_US R603
+L Device:R_US R503
 U 1 1 5E86110C
 P 4850 4400
-F 0 "R603" V 4930 4400 50  0000 C CNN
+F 0 "R503" V 4930 4400 50  0000 C CNN
 F 1 "10k" V 4770 4400 50  0000 C CNN
 F 2 "Resistor_SMD:R_0603_1608Metric" H 4850 4400 60  0001 C CNN
@@
 $EndComp
 $Comp
-L Device:R_US R601
+L Device:R_US R501
 U 1 1 5E85FF70
 P 4850 3350
-F 0 "R601" V 4930 3350 50  0000 C CNN
+F 0 "R501" V 4930 3350 50  0000 C CNN
 F 1 "10k" V 4770 3350 50  0000 C CNN
 F 2 "Resistor_SMD:R_0603_1608Metric" H 4850 3350 60  0001 C CNN
@@
 	6100 3700 6200 3700
 $Comp
-L Device:C_Small C601
+L Device:C_Small C501
 U 1 1 5E7C350B
 P 6500 3350
-F 0 "C601" H 6408 3396 50  0000 R CNN
+F 0 "C501" H 6408 3396 50  0000 R CNN
 F 1 "0.1u" H 6408 3305 50  0000 R CNN
 F 2 "Capacitor_SMD:C_0603_1608Metric" H 6500 3350 50  0001 C CNN
@@
 Connection ~ 6500 3150
 $Comp
-L power:+3.3V #PWR0601
+L power:+3.3V #PWR0501
 U 1 1 5E7A272A
 P 6500 3100
-F 0 "#PWR0601" H 6500 2950 50  0001 C CNN
+F 0 "#PWR0501" H 6500 2950 50  0001 C CNN
 F 1 "+3.3V" H 6515 3273 50  0000 C CNN
 F 2 "" H 6500 3100 50  0001 C CNN
@@
 $EndComp
 $Comp
-L Sensor_Gas:CCS811 U601
+L Sensor_Gas:CCS811 U501
 U 1 1 5E7903B2
 P 5700 3900
-F 0 "U601" H 5800 4450 50  0000 C CNN
+F 0 "U501" H 5800 4450 50  0000 C CNN
 F 1 "CCS811" H 5900 4350 50  0000 C CNN
 F 2 "Package_LGA:AMS_LGA-10-1EP_2.7x4mm_P0.6mm" H 5700 3300 50  0001 C CNN

Commit message: BOM reduction and part picking
Parts:
- R501, R502, R503: Digikey (none) -> 311-10.0KHRCT-ND; LCSC (none) -> C98220; MPN (none) -> RC0603FR-0710KL; Note (none) -> RES SMD 10K OHM 1% 1/10W 0603
Changed lines of the file:
@@
 F 2 "Resistor_SMD:R_0603_1608Metric" H 5200 3350 60  0001 C CNN
 F 3 "" H 5200 3350 60  0001 C CNN
+F 4 "311-10.0KHRCT-ND" H 5200 3350 50  0001 C CNN "Digikey"
+F 5 "C98220" H 5200 3350 50  0001 C CNN "LCSC"
+F 6 "RC0603FR-0710KL" H 5200 3350 50  0001 C CNN "MPN"
+F 7 "RES SMD 10K OHM 1% 1/10W 0603" H 5200 3350 50  0001 C CNN "Note"
 	1    5200 3350
 	1    0    0    -1
@@
 F 2 "Resistor_SMD:R_0603_1608Metric" H 4850 4400 60  0001 C CNN
 F 3 "" H 4850 4400 60  0001 C CNN
+F 4 "311-10.0KHRCT-ND" H 4850 4400 50  0001 C CNN "Digikey"
+F 5 "C98220" H 4850 4400 50  0001 C CNN "LCSC"
+F 6 "RC0603FR-0710KL" H 4850 4400 50  0001 C CNN "MPN"
+F 7 "RES SMD 10K OHM 1% 1/10W 0603" H 4850 4400 50  0001 C CNN "Note"
 	1    4850 4400
 	1    0    0    -1
@@
 F 2 "Resistor_SMD:R_0603_1608Metric" H 4850 3350 60  0001 C CNN
 F 3 "" H 4850 3350 60  0001 C CNN
+F 4 "311-10.0KHRCT-ND" H 4850 3350 50  0001 C CNN "Digikey"
+F 5 "C98220" H 4850 3350 50  0001 C CNN "LCSC"
+F 6 "RC0603FR-0710KL" H 4850 3350 50  0001 C CNN "MPN"
+F 7 "RES SMD 10K OHM 1% 1/10W 0603" H 4850 3350 50  0001 C CNN "Note"
 	1    4850 3350
 	1    0    0    -1

Commit message: Prep for gerber export
Update fields
Align standoff holes
Parts:
- U501: Manufacturer (none) -> ScioSense
Changed lines of the file:
@@
 F 5 "CCS811B-JOPR5KCT-ND" H 5700 3900 50  0001 C CNN "Digikey"
 F 6 "CCS811B-JOPR5K LGA10 LF T&R" H 5700 3900 50  0001 C CNN "Note"
+F 7 "ScioSense" H 5700 3900 50  0001 C CNN "Manufacturer"
 	1    5700 3900
 	1    0    0    -1
