File: power.sch (KiCad schematic (older format))
At the start: 39 parts, among them J801 Conn_01x02, J802 Conn_01x02, Q801 DMMT5401, Q802 DMMT5401, U801 TPS61022, U802 TLV62585, U803 MCP73831-2-OT

Commit message: BOM reduction and part picking
Parts:
- Q801: value DMMT5401 -> DMP3098L-7
- R802: LCSC (none) -> C246003
- R804, R808, R812, R813: LCSC (none) -> C98220
- R805: Digikey (none) -> 311-47.5KHRCT-ND; LCSC (none) -> C137715; MPN (none) -> RC0603FR-0747K5L; Note (none) -> RES SMD 47.5K OHM 1% 1/10W 0603
- R810, R811: LCSC (none) -> C125933
Changed lines of the file:
@@
 F 5 "311-732KHRCT-ND" H 3800 2050 50  0001 C CNN "Digikey"
 F 6 "RES SMD 732K OHM 1% 1/10W 0603" H 3800 2050 50  0001 C CNN "Note"
+F 7 "C246003" H 3800 2050 50  0001 C CNN "LCSC"
 	1    3800 2050
 	-1   0    0    1
@@
 AR Path="/5FCEDB09/5FAC6B33/5FAACE37" Ref="Q?"  Part="1"
 F 0 "Q801" V 5892 1950 50  0000 C CNN
-F 1 "DMMT5401" V 5801 1950 50  0000 C CNN
+F 1 "DMP3098L-7" V 5801 1950 50  0000 C CNN
 F 2 "Package_TO_SOT_SMD:SOT-23-6" H 5750 2050 50  0001 C CNN
 F 3 "~" H 5550 1950 50  0001 C CNN
@@
 F 5 "311-10.0KHRCT-ND" H 5100 2650 50  0001 C CNN "Digikey"
 F 6 "RES SMD 10K OHM 1% 1/10W 0603" H 5100 2650 50  0001 C CNN "Note"
+F 7 "C98220" H 5100 2650 50  0001 C CNN "LCSC"
 	1    5100 2650
 	1    0    0    -1
@@
 F 2 "Resistor_SMD:R_0603_1608Metric" H 6000 2650 60  0001 C CNN
 F 3 "" H 6000 2650 60  0001 C CNN
+F 4 "311-47.5KHRCT-ND" H 6000 2650 50  0001 C CNN "Digikey"
+F 5 " C137715 " H 6000 2650 50  0001 C CNN "LCSC"
+F 6 "RC0603FR-0747K5L" H 6000 2650 50  0001 C CNN "MPN"
+F 7 "RES SMD 47.5K OHM 1% 1/10W 0603" H 6000 2650 50  0001 C CNN "Note"
 	1    6000 2650
 	-1   0    0    1
@@
 F 7 "RES SMD 1K OHM 1% 1/10W 0603" H 8500 4450 50  0001 C CNN "Note"
 F 8 "311-1.00KHRCT-ND" H 8500 4450 50  0001 C CNN "Digikey"
-F 9 "" H 8500 4450 50  0001 C CNN "LCSC"
+F 9 "C125933" H 8500 4450 50  0001 C CNN "LCSC"
 F 10 "RC0603FR-071KL" H 8500 4450 50  0001 C CNN "MPN"
 	1    8500 4450
@@
 F 5 "311-10.0KHRCT-ND" H 7100 4200 50  0001 C CNN "Digikey"
 F 6 "RES SMD 10K OHM 1% 1/10W 0603" H 7100 4200 50  0001 C CNN "Note"
+F 7 "C98220" H 7100 4200 50  0001 C CNN "LCSC"
 	1    7100 4200
 	1    0    0    -1
@@
 F 7 "RES SMD 1K OHM 1% 1/10W 0603" H 7900 4450 50  0001 C CNN "Note"
 F 8 "311-1.00KHRCT-ND" H 7900 4450 50  0001 C CNN "Digikey"
-F 9 "" H 7900 4450 50  0001 C CNN "LCSC"
+F 9 "C125933" H 7900 4450 50  0001 C CNN "LCSC"
 F 10 "RC0603FR-071KL" H 7900 4450 50  0001 C CNN "MPN"
 	1    7900 4450
@@
 F 5 "311-10.0KHRCT-ND" H 10450 4350 50  0001 C CNN "Digikey"
 F 6 "RES SMD 10K OHM 1% 1/10W 0603" H 10450 4350 50  0001 C CNN "Note"
+F 7 "C98220" H 10450 4350 50  0001 C CNN "LCSC"
 	1    10450 4350
 	1    0    0    -1
@@
 F 5 "311-10.0KHRCT-ND" H 10450 3950 50  0001 C CNN "Digikey"
 F 6 "RES SMD 10K OHM 1% 1/10W 0603" H 10450 3950 50  0001 C CNN "Note"
+F 7 "C98220" H 10450 3950 50  0001 C CNN "LCSC"
 	1    10450 3950
 	1    0    0    -1

Commit message: Prep for gerber export
Update fields
Align standoff holes
Parts:
- U801: Manufacturer (none) -> Texas Instruments
- U802: LCSC (none) -> C485117
- U803: Manufacturer (none) -> Microchip Technology
Changed lines of the file:
@@
 F 5 "296-51694-1-ND" H 1950 3750 50  0001 C CNN "Digikey"
 F 6 "IC REG BUCK ADJUSTABLE 3A SOT563" H 1950 3750 50  0001 C CNN "Note"
+F 7 "C485117" H 1950 3750 50  0001 C CNN "LCSC"
 	1    1950 3750
 	1    0    0    -1
@@
 F 5 "296-TPS61022RWURCT-ND" H 2950 1900 50  0001 C CNN "Digikey"
 F 6 "Boost Switching Regulator IC Positive Adjustable 2.2V 1 Output  7-VFQFN" H 2950 1900 50  0001 C CNN "Note"
+F 7 "Texas Instruments" H 2950 1900 50  0001 C CNN "Manufacturer"
 	1    2950 1900
 	1    0    0    -1
@@
 F 6 "MCP73831T-2ACI/OT" H 7650 3900 50  0001 C CNN "MPN"
 F 7 "IC CONTROLLR LI-ION 4.2V SOT23-5" H 7650 3900 50  0001 C CNN "Note"
+F 8 "Microchip Technology" H 7650 3900 50  0001 C CNN "Manufacturer"
 	1    7650 3900
 	1    0    0    -1

Commit message: Schematic field cleanup
Remove stray spaces
Cleaned up duplicate fields
Normalize: 100pF (C314 C803 C807) and 47uF  (C308 C310 C804 C805) according to r0 order
Parts:
- C803, C807: Digikey 311-3351-1-ND -> 1276-1295-1-ND; LCSC (none) -> C296717; MPN CC0603GRNPO9BN101 -> CL10C101JC8NNNC; Note CAP CER 100PF 50V NPO 0603 -> CAP CER 100PF C0G 50V 0603
- C804, C805: Digikey 587-5455-1-ND -> 587-5922-1-ND; LCSC (none) -> C396815; MPN JMK325B7476MM-PR -> 1210X476K160CT; Note CAP CER 47UF 6.3V X7R 1210 -> CAP CER 47UF X5R 10V 1210; Size (none) -> 1210; Type (none) -> X5R; Voltage (none) -> 10V
- R805: LCSC C137715 -> C137715
Changed lines of the file:
@@
 F 2 "Capacitor_SMD:C_0603_1608Metric" H 2650 3850 50  0001 C CNN
 F 3 "~" H 2650 3850 50  0001 C CNN
-F 4 "CC0603GRNPO9BN101" H 2650 3850 50  0001 C CNN "MPN"
-F 5 "311-3351-1-ND" H 2650 3850 50  0001 C CNN "Digikey"
-F 6 "CAP CER 100PF 50V NPO 0603" H 2650 3850 50  0001 C CNN "Note"
+F 4 "CL10C101JC8NNNC" H 2650 3850 50  0001 C CNN "MPN"
+F 5 "1276-1295-1-ND" H 2650 3850 50  0001 C CNN "Digikey"
+F 6 "CAP CER 100PF C0G 50V 0603" H 2650 3850 50  0001 C CNN "Note"
 F 7 "1" H 2650 3850 50  0001 C CNN "DNP"
+F 8 "C296717" H 2650 3850 50  0001 C CNN "LCSC"
 	1    2650 3850
 	1    0    0    -1
@@
 F 2 "Capacitor_SMD:C_1210_3225Metric" H 4200 2050 50  0001 C CNN
 F 3 "~" H 4200 2050 50  0001 C CNN
-F 4 "JMK325B7476MM-PR" H 4200 2050 50  0001 C CNN "MPN"
-F 5 "587-5455-1-ND" H 4200 2050 50  0001 C CNN "Digikey"
-F 6 "CAP CER 47UF 6.3V X7R 1210" H 4200 2050 50  0001 C CNN "Note"
+F 4 "1210X476K160CT" H 4200 2050 50  0001 C CNN "MPN"
+F 5 "587-5922-1-ND" H 4200 2050 50  0001 C CNN "Digikey"
+F 6 "CAP CER 47UF X5R 10V 1210" H 4200 2050 50  0001 C CNN "Note"
+F 7 "C396815" H 4200 2050 50  0001 C CNN "LCSC"
+F 8 "1210" H 4200 2050 50  0001 C CNN "Size"
+F 9 "X5R" H 4200 2050 50  0001 C CNN "Type"
+F 10 "10V" H 4200 2050 50  0001 C CNN "Voltage"
 	1    4200 2050
 	1    0    0    -1
@@
 F 2 "Capacitor_SMD:C_1210_3225Metric" H 4550 2050 50  0001 C CNN
 F 3 "~" H 4550 2050 50  0001 C CNN
-F 4 "JMK325B7476MM-PR" H 4550 2050 50  0001 C CNN "MPN"
-F 5 "587-5455-1-ND" H 4550 2050 50  0001 C CNN "Digikey"
-F 6 "CAP CER 47UF 6.3V X7R 1210" H 4550 2050 50  0001 C CNN "Note"
+F 4 "1210X476K160CT" H 4550 2050 50  0001 C CNN "MPN"
+F 5 "587-5922-1-ND" H 4550 2050 50  0001 C CNN "Digikey"
+F 6 "CAP CER 47UF X5R 10V 1210" H 4550 2050 50  0001 C CNN "Note"
+F 7 "C396815" H 4550 2050 50  0001 C CNN "LCSC"
+F 8 "1210" H 4550 2050 50  0001 C CNN "Size"
+F 9 "X5R" H 4550 2050 50  0001 C CNN "Type"
+F 10 "10V" H 4550 2050 50  0001 C CNN "Voltage"
 	1    4550 2050
 	1    0    0    -1
@@
 F 2 "Capacitor_SMD:C_0603_1608Metric" H 3400 2050 50  0001 C CNN
 F 3 "~" H 3400 2050 50  0001 C CNN
-F 4 "CC0603GRNPO9BN101" H 3400 2050 50  0001 C CNN "MPN"
-F 5 "311-3351-1-ND" H 3400 2050 50  0001 C CNN "Digikey"
-F 6 "CAP CER 100PF 50V NPO 0603" H 3400 2050 50  0001 C CNN "Note"
+F 4 "CL10C101JC8NNNC" H 3400 2050 50  0001 C CNN "MPN"
+F 5 "1276-1295-1-ND" H 3400 2050 50  0001 C CNN "Digikey"
+F 6 "CAP CER 100PF C0G 50V 0603" H 3400 2050 50  0001 C CNN "Note"
+F 7 "C296717" H 3400 2050 50  0001 C CNN "LCSC"
 	1    3400 2050
 	1    0    0    -1
@@
 F 3 "" H 6000 2650 60  0001 C CNN
 F 4 "311-47.5KHRCT-ND" H 6000 2650 50  0001 C CNN "Digikey"
-F 5 " C137715 " H 6000 2650 50  0001 C CNN "LCSC"
+F 5 "C137715" H 6000 2650 50  0001 C CNN "LCSC"
 F 6 "RC0603FR-0747K5L" H 6000 2650 50  0001 C CNN "MPN"
 F 7 "RES SMD 47.5K OHM 1% 1/10W 0603" H 6000 2650 50  0001 C CNN "Note"
