File: sensor_co.sch (KiCad schematic (older format))
At the start: 10 parts, among them U601 110-102, U602 LMP91000

Commit message: BOM reduction and part picking
Parts:
- R601: value 499k -> 732k; Digikey (none) -> 311-732KHRCT-ND; LCSC (none) -> C246003; MPN (none) -> RC0603FR-07732KL; Note (none) -> RES SMD 732K OHM 1% 1/10W 0603
Changed lines of the file:
@@
 P 4350 3600
 F 0 "R601" H 4283 3646 50  0000 R CNN
-F 1 "499k" H 4283 3555 50  0000 R CNN
+F 1 "732k" H 4283 3555 50  0000 R CNN
 F 2 "Resistor_SMD:R_0603_1608Metric" H 4350 3600 50  0001 C CNN
 F 3 "~" H 4350 3600 50  0001 C CNN
+F 4 "311-732KHRCT-ND" H 4350 3600 50  0001 C CNN "Digikey"
+F 5 "C246003" H 4350 3600 50  0001 C CNN "LCSC"
+F 6 "RC0603FR-07732KL" H 4350 3600 50  0001 C CNN "MPN"
+F 7 "RES SMD 732K OHM 1% 1/10W 0603" H 4350 3600 50  0001 C CNN "Note"
 	1    4350 3600
 	1    0    0    -1

Commit message: Schematic field cleanup
Remove stray spaces
Cleaned up duplicate fields
Normalize: 100pF (C314 C803 C807) and 47uF  (C308 C310 C804 C805) according to r0 order
Parts:
- C601: Alt .1u -> (none); Current .1u -> (none); Description .1u -> (none); Error .1u -> (none); Mfr .1u -> (none)
- FB601: Mouser 81-BLM18PG471SN1D -> 81-BLM18PG471SN1D
Changed lines of the file:
@@
 F 4 "490-5223-1-ND" H 4500 3000 50  0001 C CNN "Digikey"
 F 5 "BLM18PG471SN1D" H 4500 3000 50  0001 C CNN "MPN"
-F 6 "81-BLM18PG471SN1D " H 4500 3000 50  0001 C CNN "Mouser"
+F 6 "81-BLM18PG471SN1D" H 4500 3000 50  0001 C CNN "Mouser"
 F 7 "470 Ohms @ 100MHz 1 Power Line Ferrite Bead 0603 1A 200mOhm" H 4500 3000 50  0001 C CNN "Note"
 F 8 "C97853" H 4500 3000 50  0001 C CNN "LCSC"
@@
 F 1 "0.1u" H 4592 3755 50  0000 L CNN
 F 2 "Capacitor_SMD:C_0603_1608Metric" H 4500 3800 50  0001 C CNN
-F 3 ".1u" H 4500 3800 50  0001 C CNN
+F 3 "" H 4500 3800 50  0001 C CNN
 F 4 "1292-1643-1-ND" H 4500 3800 50  0001 C CNN "Digikey"
-F 5 ".1u" H 4500 3800 50  0001 C CNN "Error"
-F 6 "" H 4500 3800 50  0001 C CNN "LCSC"
-F 7 "0603B104K500CT" H 4500 3800 50  0001 C CNN "MPN"
-F 8 "CAP CER 0.1UF 50V X7R 0603" H 4500 3800 50  0001 C CNN "Note"
-F 9 ".1u" H 4500 3800 50  0001 C CNN "Alt"
-F 10 ".1u" H 4500 3800 50  0001 C CNN "Current"
-F 11 ".1u" H 4500 3800 50  0001 C CNN "Description"
-F 12 ".1u" H 4500 3800 50  0001 C CNN "Mfr"
+F 5 "0603B104K500CT" H 4500 3800 50  0001 C CNN "MPN"
+F 6 "CAP CER 0.1UF 50V X7R 0603" H 4500 3800 50  0001 C CNN "Note"
 	1    4500 3800
 	1    0    0    -1
