File: sensor_smoke.sch (KiCad schematic (older format))
At the start: 15 parts, among them U701 TLV70018, U702 ADPD188BI, U703 Smoke Chamber

Commit message: Prep for gerber export
Update fields
Align standoff holes
Parts:
- U702: Manufacturer (none) -> Analog Devices Inc.
Changed lines of the file:
@@
 F 5 "ADPD188BI-ACEZR7" H 5400 4350 50  0001 C CNN "Digikey"
 F 6 "SENSOR SMOKE 470NM/850NM AMB 24LGA" H 5400 4350 50  0001 C CNN "Note"
+F 7 "Analog Devices Inc." H 5400 4350 50  0001 C CNN "Manufacturer"
 	1    5400 4350
 	1    0    0    -1

Commit message: Schematic field cleanup
Remove stray spaces
Cleaned up duplicate fields
Normalize: 100pF (C314 C803 C807) and 47uF  (C308 C310 C804 C805) according to r0 order
Parts:
- D701: LCSC C264281 -> C264281
- FB701: Mouser 81-BLM18PG471SN1D -> 81-BLM18PG471SN1D
Changed lines of the file:
@@
 F 5 "C97853" H 4500 2750 50  0001 C CNN "LCSC"
 F 6 "BLM18PG471SN1D" H 4500 2750 50  0001 C CNN "MPN"
-F 7 "81-BLM18PG471SN1D " H 4500 2750 50  0001 C CNN "Mouser"
+F 7 "81-BLM18PG471SN1D" H 4500 2750 50  0001 C CNN "Mouser"
 F 8 "470 Ohms @ 100MHz 1 Power Line Ferrite Bead 0603 1A 200mOhm" H 4500 2750 50  0001 C CNN "Note"
 	1    4500 2750
@@
 F 5 "1080-1140-ND" H 4450 3800 50  0001 C CNN "Digikey"
 F 6 "SENSOR PHOTODIODE 940NM RADIAL" H 4450 3800 50  0001 C CNN "Note"
-F 7 " C264281" H 4450 3800 50  0001 C CNN "LCSC"
+F 7 "C264281" H 4450 3800 50  0001 C CNN "LCSC"
 	1    4450 3800
 	0    1    1    0
