File: SD1.kicad_pcb (KiCad board)
At the start: 4 copper layers, 108 x 108 mm, 252 parts, among them J101 JST 1.25mm, J102 JST 1.25mm, J103 JST ZH 1.5mm 1x5, J201 HR861153C, J301 PJ-102AH, J302 PJ-102AH, J303 Conn_01x02, J304 Conn_01x02, J402 FTDI_TTL_Cable, J403 10118194-0001LF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

Commit message: Soldermask clearance fix
Other:
- rule pad_to_mask_clearance: 0 -> 0.0508
