File: subprojects/FLASH_MOD/FLASH_MOD.sch (KiCad schematic (older format))
At the start: 14 parts, among them U1 W25Q128JVS, U101 ER-TFTM028-4

Commit message: Flash mod add generated files
Parts:
- removed JP103: Jumper_NO_Small, Jumper:SolderJumper-2_P1.3mm_Open_RoundedPad1.0x1.5mm, symbol Device:Jumper_NO_Small
Connections:
- net labels removed: 5V_MainDet, BATT_Det, CO_ADC, DB_5V, DIO12_RXD, DIO13_TXD, DIO16_TDO, DIO17_TDI, ETH_CS, IO_INT, PIR_SENSE, RGBW_DOUT, SPKR_DRIVE, WMCU_CTS, WMCU_RESET, WMCU_RXD, WMCU_SWO, WMCU_TCK, WMCU_TMS, WMCU_TXD, WMCU_VDD, ~ETH_INT
- wire segments 74 -> 45
Other:
- note added: "Solder connections to the back of the main board"
- moved on the sheet: C1, C2, JP1, JP101, JP102, JP2, JP3, R1, TP1, TP2, U1, U101A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
